File: Hardware/KiCad/Project/SynerMycha_MKII.kicad_pcb (KiCad board)
At the start: 4 copper layers, 60 x 75 mm, 38 parts, among them J1 USB_B_Micro, J2 STDC14_STM32_JTAG_SWD, J3 B3B-XH-A, J4 B3B-XH-A, J5 Conn_01x04, J6 Conn_01x04, J7 Conn_01x04, J8 Conn_01x04, J9 Conn_01x04, Q1 IRLML9301TRPBF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

Commit message: QS
Parts:
- removed AE1: Antenna_Dipole, RF_Antenna:Texas_SWRA117D_2.4GHz_Right
- removed the SW2 at (120.0, 126.0)
- removed the SW3 at (120.0, 132.0)
- removed the SW4 at (124.0, 129.0)
- added C10: 0.1uF, Capacitor_SMD:C_0402_1005Metric, F.Cu at (218.9, 121.5)
- added C11: 10uF, Capacitor_SMD:C_0603_1608Metric, F.Cu at (199.0, 121.9)
- added C12: 0.1uF, Capacitor_SMD:C_0402_1005Metric, F.Cu at (226.5, 113.5)
- added C13: 0.1uF, Capacitor_SMD:C_0402_1005Metric, F.Cu at (222.5, 116.5)
- added C14: 10uF, Capacitor_SMD:C_0603_1608Metric, F.Cu at (223.0, 111.8)
- added C15: 0.1uF, Capacitor_SMD:C_0603_1608Metric, F.Cu at (223.0, 114.3)
- added C16: 10uF, Capacitor_SMD:C_0603_1608Metric, F.Cu at (219.7, 119.3)
- added C8: 0.1uF, Capacitor_SMD:C_0402_1005Metric, F.Cu at (226.5, 111.5)
- added C9: 10uF, Capacitor_SMD:C_0603_1608Metric, F.Cu at (195.0, 121.9)
- added J10: USB_B_Micro, Connector_USB:USB_Micro-B_Amphenol_10103594-0001LF_Horizontal, F.Cu at (126.0, 77.1)
- added J11: Conn_02x04_Odd_Even, Connector_PinSocket_2.54mm:PinSocket_2x04_P2.54mm_Horizontal, F.Cu at (131.0, 127.5)
- added Q2: S8050, Package_TO_SOT_THT:TO-92_Inline, F.Cu at (221.3, 108.0)
- added Q3: S8050, Package_TO_SOT_THT:TO-92_Inline, F.Cu at (213.2, 116.0)
- added R10: 10k, Resistor_SMD:R_0402_1005Metric, F.Cu at (216.0, 119.5)
- added R11: 10k, Resistor_SMD:R_0402_1005Metric, F.Cu at (216.0, 121.5)
- added R12: 12k, Resistor_SMD:R_0402_1005Metric, F.Cu at (216.0, 123.5)
- added R13: 12k, Resistor_SMD:R_0402_1005Metric, F.Cu at (223.2, 118.5)
- added U4: DRV8835, Package_SON:Texas_R-PWSON-N12_EP0.4x2mm, F.Cu at (218.5, 67.0)
- added U5: AS5045B, Package_SO:SSOP-16_5.3x6.2mm_P0.65mm, F.Cu at (197.8, 116.6)
- added U6: AS5045B, Package_SO:SSOP-16_5.3x6.2mm_P0.65mm, F.Cu at (197.8, 108.7)
- added U7: CP2102N-A01-GQFN28, Package_DFN_QFN:QFN-28-1EP_5x5mm_P0.5mm_EP3.35x3.35mm, F.Cu at (122.5, 84.5)
- J5, J6: footprint Connector_PinHeader_1.00mm:PinHeader_1x04_P1.00mm_Vertical -> Connector_PinHeader_1.00mm:PinHeader_1x04_P1.00mm_Horizontal
- U3: value TB6612FNG -> VL53L0X; footprint Package_SO:SSOP-24_5.3x8.2mm_P0.65mm -> VL53L0X:SENSOR_VL53L0X
- moved J9 137.0 mm to (263.5, 95.5)
- moved J5 109.7 mm to (119.5, 101.0), turned to 180 degrees
- moved SW3 107.4 mm to (208.0, 153.5), turned to 90 degrees
- moved SW4 99.0 mm to (212.5, 150.5), turned to 90 degrees
- moved SW2 98.7 mm to (212.5, 156.0), turned to 270 degrees
- moved U3 91.0 mm to (238.5, 115.5)
- moved J6 78.3 mm to (174.5, 98.0)
- moved J7 70.6 mm to (225.5, 128.5)
- moved J8 69.7 mm to (233.5, 126.5)
- moved J1 7.78 mm to (134.5, 68.5), turned to 225 degrees
Connections:
- net /D+ renamed /STM_D+
- net /D- renamed /STM_D-
- J5 pad 1: +3V3 -> /ENC_WHEEL_L_A
- J5 pad 2: /ENC_WHEEL_L_A -> /ENC_WHEEL_L_B
- J5 pad 3: /ENC_WHEEL_L_B -> GND
- J5 pad 4: GND -> +3V3
- J6 pad 2: /ENC_WHEEL_R_A -> GND
- J6 pad 4: GND -> /ENC_WHEEL_R_A
- J7 pad 1: +3V3 -> Net-(J7-Pad1)
- J7 pad 2: /ENC_WHEEL_L_A -> Net-(J7-Pad2)
- J7 pad 3: /ENC_WHEEL_L_B -> Net-(C8-Pad1)
- J7 pad 4: GND -> Net-(C8-Pad2)
- J8 pad 1: +3V3 -> Net-(J8-Pad1)
- J8 pad 2: /ENC_WHEEL_R_A -> Net-(J8-Pad2)
- J8 pad 3: /ENC_WHEEL_R_B -> Net-(C10-Pad1)
- J8 pad 4: GND -> Net-(C10-Pad2)
- U2 pad 2: /MOT_L_B -> (no net)
- U2 pad 3: /MOT_L_A -> (no net)
- U2 pad 37: /MOT_L_PWM -> (no net)
- U2 pad 38: /MOT_R_PWM -> (no net)
- U2 pad 4: /MOT_R_B -> (no net)
- U2 pad 8: /MOT_R_A -> (no net)
- U3 pad 1: Net-(U3-Pad1) -> (no net)
- U3 pad 10: GND -> (no net)
- U3 pad 11: Net-(U3-Pad11) -> (no net)
- U3 pad 12: Net-(U3-Pad11) -> Net-(U3-Pad12)
- U3 pad 2: Net-(U3-Pad1) -> (no net)
- U3 pad 3: GND -> Net-(U3-Pad12)
- U3 pad 4: GND -> Net-(U3-Pad12)
- U3 pad 5: Net-(U3-Pad5) -> (no net)
- U3 pad 6: Net-(U3-Pad5) -> Net-(U3-Pad12)
- U3 pad 7: Net-(U3-Pad7) -> (no net)
- U3 pad 8: Net-(U3-Pad7) -> (no net)
- U3 pad 9: GND -> (no net)
Routing:
- net (no net): track 65.0 -> 0.00 mm
- net Net-(U3-Pad12): track 0.00 -> 4.82 mm
Other:
- board text added: "ESP UART"
- board text added: "STM UART"
- board text removed: "OLED 0.91""

Commit message: QS
Parts:
- removed J11: Conn_02x04_Odd_Even, Connector_PinSocket_2.54mm:PinSocket_2x04_P2.54mm_Horizontal
- removed J2: STDC14_STM32_JTAG_SWD, Connector_PinHeader_1.27mm:PinHeader_2x05_P1.27mm_Vertical_SMD
- added AE2: 2.4GHz, RF_Antenna:Texas_SWRA117D_2.4GHz_Right, F.Cu at (122.5, 134.0)
- added BZ1: Buzzer, Buzzer_Beeper:Buzzer_CUI_CPT-9019S-SMT, F.Cu at (187.8, 55.2)
- added C17: 10uF, Capacitor_SMD:C_0603_1608Metric, F.Cu at (138.5, 134.5)
- added C18: 10uF, Capacitor_SMD:C_0603_1608Metric, F.Cu at (146.7, 123.1)
- added C19: 1uF, Capacitor_SMD:C_0402_1005Metric, F.Cu at (147.8, 131.3)
- added C20: 5.6pF, Capacitor_SMD:C_0402_1005Metric, F.Cu at (126.6, 129.2)
- added C21: 5.6pF, Capacitor_SMD:C_0402_1005Metric, F.Cu at (130.6, 129.2)
- added C22: 8.6pF, Capacitor_SMD:C_0402_1005Metric, F.Cu at (124.8, 133.5)
- added C23: 2.4pF, Capacitor_SMD:C_0402_1005Metric, F.Cu at (123.8, 134.5)
- added C24: 0.1uF, Capacitor_SMD:C_0603_1608Metric, F.Cu at (138.5, 132.0)
- added C25: 0.1uF, Capacitor_SMD:C_0603_1608Metric, F.Cu at (143.8, 127.2)
- added C26: 0.1uF, Capacitor_SMD:C_0603_1608Metric, F.Cu at (143.8, 129.8)
- added D1: WS2812B, LED_SMD:LED_WS2812B_PLCC4_5.0x5.0mm_P3.2mm, F.Cu at (375.0, 55.0)
- added D2: WS2812B, LED_SMD:LED_WS2812B_PLCC4_5.0x5.0mm_P3.2mm, F.Cu at (384.9, 25.3)
- added D3: WS2812B, LED_SMD:LED_WS2812B_PLCC4_5.0x5.0mm_P3.2mm, F.Cu at (375.0, 41.8)
- added D4: WS2812B, LED_SMD:LED_WS2812B_PLCC4_5.0x5.0mm_P3.2mm, F.Cu at (384.9, 31.9)
- added D5: WS2812B, LED_SMD:LED_WS2812B_PLCC4_5.0x5.0mm_P3.2mm, F.Cu at (393.3, 25.3)
- added D6: WS2812B, LED_SMD:LED_WS2812B_PLCC4_5.0x5.0mm_P3.2mm, F.Cu at (375.0, 48.4)
- added D7: WS2812B, LED_SMD:LED_WS2812B_PLCC4_5.0x5.0mm_P3.2mm, F.Cu at (384.9, 38.5)
- added D8: WS2812B, LED_SMD:LED_WS2812B_PLCC4_5.0x5.0mm_P3.2mm, F.Cu at (393.3, 31.9)
- added D9: BLUE, LED_SMD:LED_0603_1608Metric, F.Cu at (139.8, 127.9)
- added J12: Conn_01x05, Connector_PinHeader_1.00mm:PinHeader_1x05_P1.00mm_Vertical_SMD_Pin1Left, F.Cu at (382.0, 59.4)
- added J13: Conn_01x05, Connector_PinHeader_1.00mm:PinHeader_1x05_P1.00mm_Vertical_SMD_Pin1Left, F.Cu at (387.5, 45.8)
- added J14: Conn_01x05, Connector_PinHeader_1.00mm:PinHeader_1x05_P1.00mm_Vertical_SMD_Pin1Left, F.Cu at (382.0, 52.4)
- added J15: Conn_01x05, Connector_PinHeader_1.00mm:PinHeader_1x05_P1.00mm_Vertical_SMD_Pin1Left, F.Cu at (391.8, 38.7)
- added J16: Conn_01x05, Connector_PinHeader_1.00mm:PinHeader_1x05_P1.00mm_Vertical_SMD_Pin1Left, F.Cu at (382.0, 45.3)
- added J17: Conn_01x05, Connector_PinHeader_1.00mm:PinHeader_1x05_P1.00mm_Vertical_SMD_Pin1Left, F.Cu at (393.1, 45.8)
- added L1: 1.5nH, Inductor_SMD:L_0402_1005Metric, F.Cu at (123.8, 132.5)
- added R14: 10k, Resistor_SMD:R_0402_1005Metric, F.Cu at (339.9, 60.5)
- added R15: 10k, Resistor_SMD:R_0402_1005Metric, F.Cu at (337.0, 60.5)
- added R16: 10k, Resistor_SMD:R_0402_1005Metric, F.Cu at (342.8, 60.5)
- added R17: 2K2, Resistor_SMD:R_0402_1005Metric, F.Cu at (345.8, 60.5)
- added R18: 8K2, Resistor_SMD:R_0402_1005Metric, F.Cu at (348.7, 60.5)
- added R19: 2K2, Resistor_SMD:R_0402_1005Metric, F.Cu at (351.6, 60.5)
- added R20: 8K2, Resistor_SMD:R_0402_1005Metric, F.Cu at (337.0, 62.5)
- added R21: 12K, Resistor_SMD:R_0402_1005Metric, F.Cu at (144.9, 136.0)
- added R22: 12K, Resistor_SMD:R_0402_1005Metric, F.Cu at (147.8, 133.2)
- added R23: 12K, Resistor_SMD:R_0402_1005Metric, F.Cu at (147.2, 125.4)
- added R24: 12K, Resistor_SMD:R_0402_1005Metric, F.Cu at (142.0, 132.0)
- added R25: 12K, Resistor_SMD:R_0402_1005Metric, F.Cu at (147.2, 127.4)
- added R26: 12K, Resistor_SMD:R_0402_1005Metric, F.Cu at (147.2, 129.3)
- added U10: VL53L0X, VL53L0X:SENSOR_VL53L0X, F.Cu at (359.0, 70.8)
- added U11: LM317_3PinPackage, Package_TO_SOT_SMD:SOT-223, F.Cu at (375.7, 34.3)
- added U12: LM317_3PinPackage, Package_TO_SOT_SMD:SOT-223, F.Cu at (375.7, 26.1)
- added U8: VL53L0X, VL53L0X:SENSOR_VL53L0X, F.Cu at (367.0, 68.8)
- added U9: ESP-PSRAM32, Package_SO:SOIC-8_3.9x4.9mm_P1.27mm, F.Cu at (126.5, 125.0)
- added Y2: 26Mhz, 5.6pF, Crystal:Crystal_SMD_Abracon_ABM10-4Pin_2.5x2.0mm, F.Cu at (128.6, 129.2)
- U4: value DRV8835 -> ESP8266EX; footprint Package_SON:Texas_R-PWSON-N12_EP0.4x2mm -> Package_DFN_QFN:QFN-32-1EP_5x5mm_P0.5mm_EP3.45x3.45mm
- Y1: footprint Crystal:Crystal_SMD_TXC_7A-2Pin_5x3.2mm -> Crystal:Crystal_SMD_Abracon_ABM10-4Pin_2.5x2.0mm
- moved U3 127.8 mm to (360.0, 75.8), turned to 0 degrees
- moved U4 112.3 mm to (128.2, 133.8)
- moved Y1 86.8 mm to (133.0, 88.2)
Connections:
- Q2 pad 2: Net-(Q2-Pad2) -> /ESP_GPIO0
- Q3 pad 2: Net-(Q3-Pad2) -> /ESP_~RESET
- R12 pad 1: Net-(Q2-Pad2) -> /ESP_GPIO0
- R13 pad 1: Net-(Q3-Pad2) -> /ESP_~RESET
- U2 pad 46: /SWDIO -> (no net)
- U2 pad 49: /SWDCLK -> (no net)
- U2 pad 9: /MOT_NSTBY -> (no net)
- U3 pad 1: (no net) -> Net-(J13-Pad1)
- U3 pad 10: (no net) -> Net-(J13-Pad4)
- U3 pad 11: (no net) -> Net-(J13-Pad1)
- U3 pad 12: Net-(U3-Pad12) -> Net-(J13-Pad2)
- U3 pad 2: (no net) -> Net-(J13-Pad2)
- U3 pad 3: Net-(U3-Pad12) -> Net-(J13-Pad2)
- U3 pad 4: Net-(U3-Pad12) -> Net-(J13-Pad2)
- U3 pad 5: (no net) -> Net-(J13-Pad5)
- U3 pad 6: Net-(U3-Pad12) -> Net-(J13-Pad2)
- U3 pad 7: (no net) -> Net-(R14-Pad2)
- U3 pad 9: (no net) -> Net-(J13-Pad3)
- U4 pad 1: +6V -> +3V3
- U4 pad 11: /MOT_NSTBY -> +3V3
- U4 pad 12: +3V3 -> (no net)
- U4 pad 13: (no net) -> Net-(R25-Pad2)
- U4 pad 2: (no net) -> Net-(C22-Pad2)
- U4 pad 3: (no net) -> +3V3
- U4 pad 4: (no net) -> +3V3
- U4 pad 6: GND -> (no net)
- U4 pad 7: (no net) -> /ESP_EN
- U7 pad 25: (no net) -> /ESP_TX
- U7 pad 26: (no net) -> /ESP_RX
- U7 pad 29: GND -> (no net)
- Y1 pad 2: /OSC_IN -> GND
Routing:
- net Net-(U3-Pad12): track 4.82 -> 0.00 mm
- net Net-(J13-Pad2): track 0.00 -> 4.82 mm
- net Net-(AE2-Pad1): track 0.00 -> 2.56 mm
- net Net-(C22-Pad2): track 0.00 -> 2.29 mm
